Commit message: iust urdf directory for meshes

File: resources/robots/iust/urdf/iust-a1.urdf (robot description, URDF)
Before this commit: robot legs, 23 links, 22 joints
Links:
- link FL_calf: geometry collision box size=0.016 0.016 0.2; visual mesh filename=../meshes/calf.dae scale=1 1 1
- link FL_hip: geometry collision cylinder length=0.04 radius=0.046; visual mesh filename=../meshes/hip.dae scale=1 1 1
- link FL_thigh: geometry collision box size=0.043 0.034 0.22; visual mesh filename=../meshes/thigh.dae scale=1 1 1
- link FR_calf: geometry collision box size=0.016 0.016 0.2; visual mesh filename=../meshes/calf.dae scale=1 1 1
- link FR_hip: geometry collision cylinder length=0.04 radius=0.046; visual mesh filename=../meshes/hip.dae scale=1 1 1
- link FR_thigh: geometry collision box size=0.043 0.034 0.22; visual mesh filename=../meshes/thigh_mirror.dae scale=1 1 1
- link RL_calf: geometry collision box size=0.016 0.016 0.2; visual mesh filename=../meshes/calf.dae scale=1 1 1
- link RL_hip: geometry collision cylinder length=0.04 radius=0.046; visual mesh filename=../meshes/hip.dae scale=1 1 1
- link RL_thigh: geometry collision box size=0.043 0.034 0.22; visual mesh filename=../meshes/thigh.dae scale=1 1 1
- link RR_calf: geometry collision box size=0.016 0.016 0.2; visual mesh filename=../meshes/calf.dae scale=1 1 1
- link RR_hip: geometry collision cylinder length=0.04 radius=0.046; visual mesh filename=../meshes/hip.dae scale=1 1 1
- link RR_thigh: geometry collision box size=0.043 0.034 0.22; visual mesh filename=../meshes/thigh_mirror.dae scale=1 1 1
- link trunk: geometry collision box size=0.3 0.2 0.093; visual mesh filename=../meshes/trunk.dae scale=1. 1.2 1.
